Commit message: working description package

File: robot_description/urdf/components/gazebo_materials.xacro (robot description, xacro)
@@ -6,5 +6,5 @@
     <xacro:property name="lidar_color" value="Gazebo/LightBlueLaser" />
     <xacro:property name="imu_link_color" value="Gazebo/Black" />
-    <xacro:property name="wheels_link_color" value="Gazebo/Black" />
+    <xacro:property name="wheels_link_color" value="Gazebo/Red" />
     <xacro:property name="casterwheel_link_color" value="Gazebo/Blue" />
     <material name="white">

File: robot_description/urdf/components/gazebo_physics.xacro (robot description, xacro)
@@ -4,44 +4,43 @@
   <xacro:property name="caster_friction" value="0.01" />
   <xacro:property name="wheels_friction" value="1000.0" />
+  <xacro:property name="solid_object" value="100000000000000000.0" />
   <gazebo reference="base_link">
-    <mu1>${standard_friction}</mu1>
-    <mu2>${standard_friction}</mu2>
-    <selfCollide>true</selfCollide>
+    <kp>${solid_object}</kp>
+    <kd>${solid_object}</kd>
     <gravity>true</gravity>
   </gazebo>
   <gazebo reference="rightwheel_link">
+    <kp>${solid_object}</kp>
+    <kd>${solid_object}</kd>
     <mu1>${wheels_friction}</mu1>
     <mu2>${wheels_friction}</mu2>
-    <selfCollide>true</selfCollide>
   </gazebo>
   <gazebo reference="leftwheel_link">
+    <kp>${solid_object}</kp>
+    <kd>${solid_object}</kd>
     <mu1>${wheels_friction}</mu1>
     <mu2>${wheels_friction}</mu2>
-    <selfCollide>true</selfCollide>
   </gazebo>
   <gazebo reference="casterwheel_link">
+    <kp>${solid_object}</kp>
+    <kd>${solid_object}</kd>
     <mu1>${caster_friction}</mu1>
     <mu2>${caster_friction}</mu2>
-    <selfCollide>true</selfCollide>
   </gazebo>
   <gazebo reference="lidar_link">
-    <mu1>${standard_friction}</mu1>
-    <mu2>${standard_friction}</mu2>
-    <selfCollide>true</selfCollide>
+    <kp>${solid_object}</kp>
+    <kd>${solid_object}</kd>
   </gazebo>
   <gazebo reference="camerad435i_link">
-    <mu1>${standard_friction}</mu1>
-    <mu2>${standard_friction}</mu2>
-    <selfCollide>true</selfCollide>
+    <kp>${solid_object}</kp>
+    <kd>${solid_object}</kd>
   </gazebo>
   <gazebo reference="camerat265_link">
-    <mu1>${standard_friction}</mu1>
-    <mu2>${standard_friction}</mu2>
-    <selfCollide>true</selfCollide>
+    <kp>${solid_object}</kp>
+    <kd>${solid_object}</kd>
   </gazebo>
   <gazebo reference="imu_link">
-    <mu1>${standard_friction}</mu1>
-    <mu2>${standard_friction}</mu2>
-    <selfCollide>true</selfCollide>
+    <kp>${solid_object}</kp>
+    <kd>${solid_object}</kd>
   </gazebo>
 </robot>

File: robot_description/urdf/robot.urdf.xacro (robot description, xacro)
@@ -3,5 +3,5 @@
     <!-- Example link -->
     <xacro:include filename="robot_core.xacro"/>
-    <xacro:include filename="$(find robot_description)/urdf/components/gazebo_control.xacro"/>
+    <!-- <xacro:include filename="$(find robot_description)/urdf/components/gazebo_control.xacro"/> -->
     <!-- <xacro:generic_laser>
         <xacro:insert_block name="laser_pose" />

File: robot_description/urdf/robot_core.xacro (robot description, xacro)
@@ -11,4 +11,6 @@
     <xacro:include filename="$(find robot_description)/sensors/depth_sensor.urdf.xacro" /> -->
     <xacro:property name="scale_ratio" value="1" />
+    <!-- Path Meshes -->
+    <xacro:property name="path_meshes" value="file://$(find robot_description)/urdf/meshes" />
     <!-- ****************** Robot bases ***************************  -->
     <!-- Define the center of the main robot chassis projected on the ground -->
@@ -21,5 +23,5 @@
             <geometry>
                 <mesh scale="${scale_ratio} ${scale_ratio} ${scale_ratio}"
-                    filename="file://$(find robot_description)/urdf/meshes/base_link.STL" />
+                    filename="${path_meshes}/base_link.stl" />
             </geometry>
             <material name="white">
@@ -27,8 +29,7 @@
         </visual>
         <collision>
-            <origin xyz="0 0 0" rpy="0 0 0" />
-            <geometry>
-                <mesh scale="${scale_ratio} ${scale_ratio} ${scale_ratio}"
-                    filename="file://$(find robot_description)/urdf/meshes/base_link.STL" />
+            <origin xyz="0.02 0 0.1" rpy="0 0 0" />
+            <geometry>
+                <box size="0.5 0.345 0.377971" />
             </geometry>
         </collision>
@@ -41,13 +42,13 @@
         <parent link="base_footprint" />
         <child link="base_link" />
-        <origin xyz="0 0 -0.14" rpy="0 0 0" />
+        <origin xyz="0 0 1" rpy="0 0 0" />
     </joint>
     <!-- Right Wheel -->
     <link name="rightwheel_link">
         <visual>
-            <origin xyz="0 0 0" rpy="0 0 0" />
-            <geometry>
-                <mesh scale="${scale_ratio} ${scale_ratio} ${scale_ratio}"
-                    filename="file://$(find robot_description)/urdf/meshes/rightwheel.STL" />
+            <origin xyz="0 0 0" rpy="3.14 0 0" />
+            <geometry>
+                <mesh scale="0.01 0.01 0.01"
+                    filename="${path_meshes}/rightwheel1.stl" />
             </geometry>
             <material name="black">
@@ -55,8 +56,7 @@
         </visual>
         <collision>
-            <origin xyz="0 0 0" rpy="0 0 0" />
-            <geometry>
-                <mesh scale="${scale_ratio} ${scale_ratio} ${scale_ratio}"
-                    filename="file://$(find robot_description)/urdf/meshes/rightwheel.STL" />
+            <origin xyz="0 0.03 0" rpy="1.5708 0 0" />
+            <geometry>
+                <cylinder radius="0.082" length="0.06"/>
             </geometry>
         </collision>
@@ -67,16 +67,16 @@
     <!-- Right Wheel Joint -->
     <joint name="rightwheel_joint" type="continuous">
-        <origin xyz="-0.12418 0.185 -0.063" rpy="0 0 3.1416" />
+        <origin xyz="-0.12418 0.185 -0.063" rpy="0 0 0" />
         <parent link="base_link" />
         <child link="rightwheel_link" />
-        <axis xyz="0 1 0" />
+        <axis xyz="0 -1 0" />
     </joint>
     <!-- Left Wheel -->
     <link name="leftwheel_link">
         <visual>
-            <origin xyz="0 0 0" rpy="0 0 0" />
-            <geometry>
-                <mesh scale="${scale_ratio} ${scale_ratio} ${scale_ratio}"
-                    filename="file://$(find robot_description)/urdf/meshes/leftwheel.STL" />
+            <origin xyz="0 0 0" rpy="3.14 0 0" />
+            <geometry>
+                <mesh scale="0.01 0.01 0.01"
+                    filename="${path_meshes}/rightwheel1.stl" />
             </geometry>
             <material name="black">
@@ -84,8 +84,7 @@
         </visual>
         <collision>
-            <origin xyz="0 0 0" rpy="0 0 0" />
-            <geometry>
-                <mesh scale="${scale_ratio} ${scale_ratio} ${scale_ratio}"
-                    filename="file://$(find robot_description)/urdf/meshes/leftwheel.STL" />
+            <origin xyz="0 0.03 0" rpy="1.5708 0 0" />
+            <geometry>
+                <cylinder radius="0.082" length="0.06"/>
             </geometry>
         </collision>
@@ -107,5 +106,5 @@
             <geometry>
                 <mesh scale="${scale_ratio} ${scale_ratio} ${scale_ratio}"
-                    filename="file://$(find robot_description)/urdf/meshes/casterwheel.STL" />
+                    filename="${path_meshes}/casterwheel.stl" />
             </geometry>
             <material name="blue">
@@ -113,8 +112,7 @@
         </visual>
         <collision>
-            <origin xyz="0 0 0" rpy="0 0 0" />
-            <geometry>
-                <mesh scale="${scale_ratio} ${scale_ratio} ${scale_ratio}"
-                    filename="file://$(find robot_description)/urdf/meshes/casterwheel.STL" />
+            <origin xyz="0 0 0" rpy="1.5708 0 0" />
+            <geometry>
+                <cylinder radius="0.04" length="0.02"/>
             </geometry>
         </collision>
@@ -125,5 +123,5 @@
     <!-- Caster Wheel Joint -->
     <joint name="casterwheel_joint" type="fixed">
-        <origin xyz="0.25029 -0.01098 -0.1075" rpy="0 0 0" />
+        <origin xyz="0.25029 -0.01098 -0.1375" rpy="0 0 0" />
         <parent link="base_link" />
         <child link="casterwheel_link" />
@@ -131,16 +129,10 @@
     </joint>
     <!-- Lidar -->
-    <link name="lidar_link">
-        <inertial>
-            <origin xyz="0.00050486 -3.7855E-05 -0.025753" rpy="0 0 0" />
-            <mass value="0.2064" />
-            <inertia ixx="0.00011156" ixy="-1.2701E-07" ixz="-1.6019E-06" iyy="0.00010988"
-                iyz="1.201E-07" izz="0.0001391" />
-        </inertial>
-        <visual>
-            <origin xyz="0 0 0" rpy="0 0 0" />
-            <geometry>
-                <mesh scale="${scale_ratio} ${scale_ratio} ${scale_ratio}"
-                    filename="file://$(find robot_description)/urdf/meshes/lidar.STL" />
+    <!-- <link name="lidar_link">
+        <visual>
+            <origin xyz="0 0 0" rpy="0 0 0" />
+            <geometry>
+                <mesh scale="${scale_ratio} ${scale_ratio} ${scale_ratio}"
+                    filename="${path_meshes}/lidar.STL" />
             </geometry>
             <material name="gray">
@@ -151,5 +143,5 @@
             <geometry>
                 <mesh scale="${scale_ratio} ${scale_ratio} ${scale_ratio}"
-                    filename="file://$(find robot_description)/urdf/meshes/lidar.STL" />
+                    filename="${path_meshes}/lidar.STL" />
             </geometry>
         </collision>
@@ -157,25 +149,19 @@
             <origin xyz="0.00050486 -3.7855E-05 -0.025753" rpy="0 0 0" />
         </xacro:inertial_box>
-    </link>
+    </link> -->
     <!-- Lidar Joint -->
-    <joint name="lidar_joint" type="fixed">
+    <!-- <joint name="lidar_joint" type="fixed">
         <origin xyz="0.00082049 0.00875 0.12332" rpy="0 0 0" />
         <parent link="base_link" />
         <child link="lidar_link" />
         <axis xyz="0 0 1" />
-    </joint>
+    </joint> -->
     <!-- IMU -->
-    <link name="imu_link">
-        <inertial>
-            <origin xyz="-0.015015 -0.00012812 0.00021369" rpy="0 0 0" />
-            <mass value="0.05157" />
-            <inertia ixx="1.5728E-05" ixy="-1.2026E-09" ixz="1.5815E-09" iyy="8.9379E-06"
-                iyz="-2.1887E-10" izz="1.4344E-05" />
-        </inertial>
-        <visual>
-            <origin xyz="0 0 0" rpy="0 0 0" />
-            <geometry>
-                <mesh scale="${scale_ratio} ${scale_ratio} ${scale_ratio}"
-                    filename="file://$(find robot_description)/urdf/meshes/imu.STL" />
+    <!-- <link name="imu_link">
+        <visual>
+            <origin xyz="0 0 0" rpy="0 0 0" />
+            <geometry>
+                <mesh scale="${scale_ratio} ${scale_ratio} ${scale_ratio}"
+                    filename="${path_meshes}/imu.STL" />
             </geometry>
             <material name="black">
@@ -186,5 +172,5 @@
             <geometry>
                 <mesh scale="${scale_ratio} ${scale_ratio} ${scale_ratio}"
-                    filename="file://$(find robot_description)/urdf/meshes/imu.STL" />
+                    filename="${path_meshes}/imu.STL" />
             </geometry>
         </collision>
@@ -192,25 +178,19 @@
             <origin xyz="-0.015015 -0.00012812 0.00021369" rpy="0 0 0" />
         </xacro:inertial_box>
-    </link>
+    </link> -->
     <!-- IMU Joint -->
-    <joint name="imu_joint" type="fixed">
+    <!-- <joint name="imu_joint" type="fixed">
         <origin xyz="0.05082 -0.0047896 0.053918" rpy="0 0 0" />
         <parent link="base_link" />
         <child link="imu_link" />
         <axis xyz="0 0 0" />
-    </joint>
+    </joint> -->
     <!-- Camera -->
-    <link name="camerad435i_link">
-        <inertial>
-            <origin xyz="0.0094812 3.7095E-05 -7.9734E-05" rpy="0 0 0" />
-            <mass value="0.032264" />
-            <inertia ixx="2.2098E-05" ixy="-1.4651E-10" ixz="2.902E-10" iyy="1.9467E-06"
-                iyz="8.3417E-11" izz="2.1858E-05" />
-        </inertial>
-        <visual>
-            <origin xyz="0 0 0" rpy="0 0 0" />
-            <geometry>
-                <mesh scale="${scale_ratio} ${scale_ratio} ${scale_ratio}"
-                    filename="file://$(find robot_description)/urdf/meshes/camerad435i.STL" />
+    <!-- <link name="camerad435i_link">
+        <visual>
+            <origin xyz="0 0 0" rpy="0 0 0" />
+            <geometry>
+                <mesh scale="${scale_ratio} ${scale_ratio} ${scale_ratio}"
+                    filename="${path_meshes}/camerad435i.STL" />
             </geometry>
             <material name="white">
@@ -221,5 +201,5 @@
             <geometry>
                 <mesh scale="${scale_ratio} ${scale_ratio} ${scale_ratio}"
-                    filename="file://$(find robot_description)/urdf/meshes/camerad435i.STL" />
+                    filename="${path_meshes}/camerad435i.STL" />
             </geometry>
         </collision>
@@ -227,25 +207,19 @@
             <origin xyz="0.0094812 3.7095E-05 -7.9734E-05" rpy="0 0 0" />
         </xacro:inertial_box>
-    </link>
+    </link> -->
     <!-- Camera Joint -->
-    <joint name="camerad435i_joint" type="fixed">
+    <!-- <joint name="camerad435i_joint" type="fixed">
         <origin xyz="-0.20718 -0.08268 0.17016" rpy="0 0 0" />
         <parent link="base_link" />
         <child link="camerad435i_link" />
         <axis xyz="0 0 0" />
-    </joint>
+    </joint> -->
     <!-- Camera -->
-    <link name="camerat265_link">
-        <inertial>
-            <origin xyz="0.0061266 3.8568E-05 -1.9004E-05" rpy="0 0 0" />
-            <mass value="0.030988" />
-            <inertia ixx="3.0221E-05" ixy="-1.6541E-10" ixz="4.8935E-11" iyy="1.9363E-06"
-                iyz="9.2265E-11" izz="2.9002E-05" />
-        </inertial>
-        <visual>
-            <origin xyz="0 0 0" rpy="0 0 0" />
-            <geometry>
-                <mesh scale="${scale_ratio} ${scale_ratio} ${scale_ratio}"
-                    filename="file://$(find robot_description)/urdf/meshes/camerat265.STL" />
+    <!-- <link name="camerat265_link">
+        <visual>
+            <origin xyz="0 0 0" rpy="0 0 0" />
+            <geometry>
+                <mesh scale="${scale_ratio} ${scale_ratio} ${scale_ratio}"
+                    filename="${path_meshes}/camerat265.STL" />
             </geometry>
             <material name="white">
@@ -256,5 +230,5 @@
             <geometry>
                 <mesh scale="${scale_ratio} ${scale_ratio} ${scale_ratio}"
-                    filename="file://$(find robot_description)/urdf/meshes/camerat265.STL" />
+                    filename="${path_meshes}/camerat265.STL" />
             </geometry>
         </collision>
@@ -262,11 +236,11 @@
             <origin xyz="0.0061266 3.8568E-05 -1.9004E-05" rpy="0 0 0" />
         </xacro:inertial_box>
-    </link>
+    </link> -->
     <!-- Camera Joint -->
-    <joint name="camerat265_joint" type="fixed">
+    <!-- <joint name="camerat265_joint" type="fixed">
         <origin xyz="-0.20118 0.080908 0.16952" rpy="0 0 0" />
         <parent link="base_link" />
         <child link="camerat265_link" />
         <axis xyz="0 0 0" />
-    </joint>
+    </joint> -->
 </robot>
