Commit message: added gazebo & bridge

File: robot_description/urdf/components/gazebo_control.xacro (robot description, xacro)
@@ -3,30 +3,38 @@
     xmlns:xacro="http://www.ros.org/wiki/xacro">
 <gazebo>
-    <plugin name="ignition::gazebo::systems::DiffDrive" filename="libignition-gazebo-diff-drive-system.so">
-        <left_joint>leftwheel_joint</left_joint>
-        <right_joint>rightwheel_joint</right_joint>
-        <wheel_separation>0.255</wheel_separation>
-        <wheel_diameter>0.066</wheel_diameter>
-        <!--limits-->
-        <max_wheel_torque>200</max_wheel_torque>
-        <max_wheel_acceleration>10.0</max_wheel_acceleration>
-        <!--outputs-->
-        <odometry_frame>odom</odometry_frame>
-        <robot_base_frame>base_footprint</robot_base_frame>
-        <publish_wheel_tf>true</publish_wheel_tf>
-        <publish_odom_tf>true</publish_odom_tf>
-        <publish_odom>false</publish_odom>
-        <publish_wheel_joint_state>true</publish_wheel_joint_state>
-        <topic>cmd_vel</topic>
+    <plugin
+        filename="gz-sim-diff-drive-system"
+        name="gz::sim::systems::DiffDrive">
+        <left_joint>left_wheel_joint</left_joint>
+        <right_joint>right_wheel_joint</right_joint>
+        <wheel_separation>0.35</wheel_separation>
+        <wheel_radius>0.05</wheel_radius>
+        <odom_publish_frequency>1</odom_publish_frequency>
+        <max_linear_acceleration>1</max_linear_acceleration>
+        <min_linear_acceleration>-1</min_linear_acceleration>
+        <max_angular_acceleration>2</max_angular_acceleration>
+        <min_angular_acceleration>-2</min_angular_acceleration>
+        <max_linear_velocity>0.5</max_linear_velocity>
+        <min_linear_velocity>-0.5</min_linear_velocity>
+        <max_angular_velocity>1</max_angular_velocity>
+        <min_angular_velocity>-1</min_angular_velocity>
     </plugin>
-    <!-- <plugin name='joint_state_publisher' filename='libgazebo_ros_joint_state_publisher.so'>
-        <jointName>leftwheel_joint</jointName>
-        <jointName>rightwheel_joint</jointName>
-        <update_rate>50.0</update_rate>
-        <alwaysOn>true</alwaysOn>
-    </plugin> -->
-    <!-- Joint states plugin -->
-    <plugin name="ignition::gazebo::systems::JointStatePublisher"
-        filename="libignition-gazebo-joint-state-publisher-system.so">
+    <plugin
+        filename="gz-sim-joint-state-publisher-system"
+        name="gz::sim::systems::JointStatePublisher">
+    </plugin>
+    <plugin
+        filename="gz-sim-pose-publisher-system"
+        name="gz::sim::systems::PosePublisher">
+        <publish_link_pose>true</publish_link_pose>
+        <use_pose_vector_msg>true</use_pose_vector_msg>
+        <static_publisher>true</static_publisher>
+        <static_update_frequency>1</static_update_frequency>
+    </plugin>
+    <plugin
+        filename="gz-sim-odometry-publisher-system"
+        name="gz::sim::systems::OdometryPublisher">
+        <odom_frame>diff_drive/odom</odom_frame>
+        <robot_base_frame>base_link</robot_base_frame>
     </plugin>
 </gazebo>

File: robot_description/urdf/robot.urdf.xacro (robot description, xacro)
@@ -2,5 +2,5 @@
 <robot xmlns:xacro="http://www.ros.org/wiki/xacro"  name="MTT_robot">
     <!-- Example link -->
-    <xacro:include filename="robot_core.xacro"/>
+    <xacro:include filename="robot_core2.xacro"/>
     <!-- <xacro:include filename="$(find robot_description)/urdf/components/gazebo_control.xacro"/> -->
     <!-- <xacro:generic_laser>

File: robot_description/urdf/robot_core.xacro (robot description, xacro)
@@ -6,8 +6,9 @@
     <xacro:include filename="$(find robot_description)/urdf/components/inertial_macros.xacro" />
     <xacro:include filename="$(find robot_description)/urdf/components/gazebo_materials.xacro" />
-    <xacro:include filename="$(find robot_description)/urdf/components/gazebo_physics.xacro" />
+    <!-- <xacro:include filename="$(find robot_description)/urdf/components/gazebo_physics.xacro" /> -->
     <!-- Sensors -->
     <!-- <xacro:include filename="$(find robot_description)/sensors/generic_laser.urdf.xacro" />
     <xacro:include filename="$(find robot_description)/sensors/depth_sensor.urdf.xacro" /> -->
+    <xacro:property name="M_PI" value="3.14159"/>
     <xacro:property name="scale_ratio" value="1" />
     <!-- Path Meshes -->
@@ -21,17 +22,20 @@
         <visual>
             <origin xyz="0 0 0" rpy="0 0 0" />
-            <geometry>
+            <!-- <geometry>
                 <mesh scale="${scale_ratio} ${scale_ratio} ${scale_ratio}"
                     filename="${path_meshes}/base_link.stl" />
+            </geometry> -->
+            <geometry>
+                <box size="0.5 0.345 0.377971" />
             </geometry>
             <material name="white">
             </material>
         </visual>
-        <collision>
+        <!-- <collision>
             <origin xyz="0.02 0 0.1" rpy="0 0 0" />
             <geometry>
                 <box size="0.5 0.345 0.377971" />
             </geometry>
-        </collision>
+        </collision> -->
         <xacro:inertial_box mass="5.79174328389446" x="-0.0374777931065171"
             y="-0.000742607274570373" z="0.0517646177576365">
@@ -47,18 +51,21 @@
     <link name="rightwheel_link">
         <visual>
-            <origin xyz="0 0 0" rpy="3.14 0 0" />
-            <geometry>
+            <origin xyz="0 0 0" rpy="0 0 0" />
+            <!-- <geometry>
                 <mesh scale="0.01 0.01 0.01"
                     filename="${path_meshes}/rightwheel1.stl" />
+            </geometry> -->
+            <geometry>
+                <cylinder radius="0.082" length="0.06"/>
             </geometry>
             <material name="black">
             </material>
         </visual>
-        <collision>
+        <!-- <collision>
             <origin xyz="0 0.03 0" rpy="1.5708 0 0" />
             <geometry>
                 <cylinder radius="0.082" length="0.06"/>
             </geometry>
-        </collision>
+        </collision> -->
         <xacro:inertial_box mass="1.0582" x="-1.2143E-17" y="0.033904" z="1.3878E-17">
             <origin xyz="-1.2143E-17 0.033904 1.3878E-17" rpy="0 0 0" />
@@ -67,26 +74,29 @@
     <!-- Right Wheel Joint -->
     <joint name="rightwheel_joint" type="continuous">
-        <origin xyz="-0.12418 0.185 -0.063" rpy="0 0 0" />
+        <origin xyz="-0.12418 0.185 -0.063" rpy="-${M_PI/2} 0 0" />
         <parent link="base_link" />
         <child link="rightwheel_link" />
-        <axis xyz="0 -1 0" />
+        <axis xyz="0 0 -1" />
     </joint>
     <!-- Left Wheel -->
     <link name="leftwheel_link">
         <visual>
-            <origin xyz="0 0 0" rpy="3.14 0 0" />
-            <geometry>
+            <origin xyz="0 0 0" rpy="0 0 0" />
+            <!-- <geometry>
                 <mesh scale="0.01 0.01 0.01"
                     filename="${path_meshes}/rightwheel1.stl" />
+            </geometry> -->
+            <geometry>
+                <cylinder radius="0.082" length="0.06"/>
             </geometry>
             <material name="black">
             </material>
         </visual>
-        <collision>
+        <!-- <collision>
             <origin xyz="0 0.03 0" rpy="1.5708 0 0" />
             <geometry>
                 <cylinder radius="0.082" length="0.06"/>
             </geometry>
-        </collision>
+        </collision> -->
         <xacro:inertial_box mass="1.0582" x="-2.4286E-17" y="-0.033904" z="4.1633E-17">
             <origin xyz="-2.4286E-17 -0.033904 4.1633E-17" rpy="0 0 0" />
@@ -95,8 +105,8 @@
     <!-- Left Wheel Joint -->
     <joint name="leftwheel_joint" type="continuous">
-        <origin xyz="-0.12418 -0.185 -0.063" rpy="0 0 -3.1416" />
+        <origin xyz="-0.12418 -0.185 -0.063" rpy="-${M_PI/2} 0 0" />
         <parent link="base_link" />
         <child link="leftwheel_link" />
-        <axis xyz="0 1 0" />
+        <axis xyz="0 0 1" />
     </joint>
     <!-- Caster Wheel -->
@@ -104,17 +114,20 @@
         <visual>
             <origin xyz="0 0 0" rpy="0 0 0" />
-            <geometry>
+            <!-- <geometry>
                 <mesh scale="${scale_ratio} ${scale_ratio} ${scale_ratio}"
                     filename="${path_meshes}/casterwheel.stl" />
+            </geometry> -->
+            <geometry>
+                <cylinder radius="0.04" length="0.02"/>
             </geometry>
             <material name="blue">
             </material>
         </visual>
-        <collision>
+        <!-- <collision>
             <origin xyz="0 0 0" rpy="1.5708 0 0" />
             <geometry>
                 <cylinder radius="0.04" length="0.02"/>
             </geometry>
-        </collision>
+        </collision> -->
         <xacro:inertial_box mass="0.10255" x="-0.0032546" y="0.0053327" z="0.013127">
             <origin xyz="-0.0032546 0.0053327 0.013127" rpy="0 0 0" />
