Commit message: Feat/simulator (#4)
* fix: dev container x11 issue

* refactor: rviz2 panel updated

* fix: rviz & gazebo plugins

* feat:  robot_worlds pkg added

* fix: tasks

* feat: ros ign bridge launch

* feat: cmake

* feat: gazebo launch

* fix: position params

* feat: use sim time

* updated docker image in dev container

* working description package

* added gazebo & bridge

* fixed lint errors

* disable cpp check no pkg now

File: robot_description/urdf/components/gazebo_control.xacro (robot description, xacro)
@@ -1,19 +1,40 @@
 <?xml version="1.0"?>
-<robot xmlns:xacro="http://www.ros.org/wiki/xacro">
+<robot name="robot_wheels"
+    xmlns:xacro="http://www.ros.org/wiki/xacro">
 <gazebo>
-    <plugin name="diff_drive" filename="libgazebo_ros_diff_drive.so">
+    <plugin
+        filename="gz-sim-diff-drive-system"
+        name="gz::sim::systems::DiffDrive">
         <left_joint>left_wheel_joint</left_joint>
         <right_joint>right_wheel_joint</right_joint>
-        <wheel_separation>0.255</wheel_separation>
-        <wheel_diameter>0.066</wheel_diameter>
-        <!--limits-->
-        <max_wheel_torque>200</max_wheel_torque>
-        <max_wheel_acceleration>10.0</max_wheel_acceleration>
-        <!--outputs-->
-        <odometry_frame>odom</odometry_frame>
-        <robot_base_frame>base_footprint</robot_base_frame>
-        <publish_wheel_tf>true</publish_wheel_tf>
-        <publish_odom_tf>true</publish_odom_tf>
-        <publish_odom>false</publish_odom>
+        <wheel_separation>0.35</wheel_separation>
+        <wheel_radius>0.05</wheel_radius>
+        <odom_publish_frequency>1</odom_publish_frequency>
+        <max_linear_acceleration>1</max_linear_acceleration>
+        <min_linear_acceleration>-1</min_linear_acceleration>
+        <max_angular_acceleration>2</max_angular_acceleration>
+        <min_angular_acceleration>-2</min_angular_acceleration>
+        <max_linear_velocity>0.5</max_linear_velocity>
+        <min_linear_velocity>-0.5</min_linear_velocity>
+        <max_angular_velocity>1</max_angular_velocity>
+        <min_angular_velocity>-1</min_angular_velocity>
+    </plugin>
+    <plugin
+        filename="gz-sim-joint-state-publisher-system"
+        name="gz::sim::systems::JointStatePublisher">
+    </plugin>
+    <plugin
+        filename="gz-sim-pose-publisher-system"
+        name="gz::sim::systems::PosePublisher">
+        <publish_link_pose>true</publish_link_pose>
+        <use_pose_vector_msg>true</use_pose_vector_msg>
+        <static_publisher>true</static_publisher>
+        <static_update_frequency>1</static_update_frequency>
+    </plugin>
+    <plugin
+        filename="gz-sim-odometry-publisher-system"
+        name="gz::sim::systems::OdometryPublisher">
+        <odom_frame>diff_drive/odom</odom_frame>
+        <robot_base_frame>base_link</robot_base_frame>
     </plugin>
 </gazebo>

File: robot_description/urdf/robot.urdf.xacro (robot description, xacro)
@@ -1,7 +1,7 @@
 <?xml version="1.0"?>
-<robot xmlns:xacro="http://www.ros.org/wiki/xacro"  name="robot">
+<robot xmlns:xacro="http://www.ros.org/wiki/xacro"  name="MTT_robot">
     <!-- Example link -->
-    <xacro:include filename="robot_core.xacro"/>
-    <xacro:include filename="$(find robot_description)/urdf/components/gazebo_control.xacro"/>
+    <xacro:include filename="robot_core2.xacro"/>
+    <!-- <xacro:include filename="$(find robot_description)/urdf/components/gazebo_control.xacro"/> -->
     <!-- <xacro:generic_laser>
         <xacro:insert_block name="laser_pose" />

File: robot_description/urdf/robot_core.xacro (robot description, xacro)
@@ -6,9 +6,12 @@
     <xacro:include filename="$(find robot_description)/urdf/components/inertial_macros.xacro" />
     <xacro:include filename="$(find robot_description)/urdf/components/gazebo_materials.xacro" />
-    <xacro:include filename="$(find robot_description)/urdf/components/gazebo_physics.xacro" />
+    <!-- <xacro:include filename="$(find robot_description)/urdf/components/gazebo_physics.xacro" /> -->
     <!-- Sensors -->
     <!-- <xacro:include filename="$(find robot_description)/sensors/generic_laser.urdf.xacro" />
     <xacro:include filename="$(find robot_description)/sensors/depth_sensor.urdf.xacro" /> -->
+    <xacro:property name="M_PI" value="3.14159"/>
     <xacro:property name="scale_ratio" value="1" />
+    <!-- Path Meshes -->
+    <xacro:property name="path_meshes" value="file://$(find robot_description)/urdf/meshes" />
     <!-- ****************** Robot bases ***************************  -->
     <!-- Define the center of the main robot chassis projected on the ground -->
@@ -19,18 +22,20 @@
         <visual>
             <origin xyz="0 0 0" rpy="0 0 0" />
-            <geometry>
-                <mesh scale="${scale_ratio} ${scale_ratio} ${scale_ratio}"
-                    filename="file://$(find robot_description)/urdf/meshes/base_link.STL" />
+            <!-- <geometry>
+                <mesh scale="${scale_ratio} ${scale_ratio} ${scale_ratio}"
+                    filename="${path_meshes}/base_link.stl" />
+            </geometry> -->
+            <geometry>
+                <box size="0.5 0.345 0.377971" />
             </geometry>
             <material name="white">
             </material>
         </visual>
-        <collision>
-            <origin xyz="0 0 0" rpy="0 0 0" />
-            <geometry>
-                <mesh scale="${scale_ratio} ${scale_ratio} ${scale_ratio}"
-                    filename="file://$(find robot_description)/urdf/meshes/base_link.STL" />
-            </geometry>
-        </collision>
+        <!-- <collision>
+            <origin xyz="0.02 0 0.1" rpy="0 0 0" />
+            <geometry>
+                <box size="0.5 0.345 0.377971" />
+            </geometry>
+        </collision> -->
         <xacro:inertial_box mass="5.79174328389446" x="-0.0374777931065171"
             y="-0.000742607274570373" z="0.0517646177576365">
@@ -41,5 +46,5 @@
         <parent link="base_footprint" />
         <child link="base_link" />
-        <origin xyz="0 0 -0.14" rpy="0 0 0" />
+        <origin xyz="0 0 1" rpy="0 0 0" />
     </joint>
     <!-- Right Wheel -->
@@ -47,18 +52,20 @@
         <visual>
             <origin xyz="0 0 0" rpy="0 0 0" />
-            <geometry>
-                <mesh scale="${scale_ratio} ${scale_ratio} ${scale_ratio}"
-                    filename="file://$(find robot_description)/urdf/meshes/rightwheel.STL" />
+            <!-- <geometry>
+                <mesh scale="0.01 0.01 0.01"
+                    filename="${path_meshes}/rightwheel1.stl" />
+            </geometry> -->
+            <geometry>
+                <cylinder radius="0.082" length="0.06"/>
             </geometry>
             <material name="black">
             </material>
         </visual>
-        <collision>
-            <origin xyz="0 0 0" rpy="0 0 0" />
-            <geometry>
-                <mesh scale="${scale_ratio} ${scale_ratio} ${scale_ratio}"
-                    filename="file://$(find robot_description)/urdf/meshes/rightwheel.STL" />
-            </geometry>
-        </collision>
+        <!-- <collision>
+            <origin xyz="0 0.03 0" rpy="1.5708 0 0" />
+            <geometry>
+                <cylinder radius="0.082" length="0.06"/>
+            </geometry>
+        </collision> -->
         <xacro:inertial_box mass="1.0582" x="-1.2143E-17" y="0.033904" z="1.3878E-17">
             <origin xyz="-1.2143E-17 0.033904 1.3878E-17" rpy="0 0 0" />
@@ -67,8 +74,8 @@
     <!-- Right Wheel Joint -->
     <joint name="rightwheel_joint" type="continuous">
-        <origin xyz="-0.12418 0.185 -0.063" rpy="0 0 3.1416" />
+        <origin xyz="-0.12418 0.185 -0.063" rpy="-${M_PI/2} 0 0" />
         <parent link="base_link" />
         <child link="rightwheel_link" />
-        <axis xyz="0 1 0" />
+        <axis xyz="0 0 -1" />
     </joint>
     <!-- Left Wheel -->
@@ -76,18 +83,20 @@
         <visual>
             <origin xyz="0 0 0" rpy="0 0 0" />
-            <geometry>
-                <mesh scale="${scale_ratio} ${scale_ratio} ${scale_ratio}"
-                    filename="file://$(find robot_description)/urdf/meshes/leftwheel.STL" />
+            <!-- <geometry>
+                <mesh scale="0.01 0.01 0.01"
+                    filename="${path_meshes}/rightwheel1.stl" />
+            </geometry> -->
+            <geometry>
+                <cylinder radius="0.082" length="0.06"/>
             </geometry>
             <material name="black">
             </material>
         </visual>
-        <collision>
-            <origin xyz="0 0 0" rpy="0 0 0" />
-            <geometry>
-                <mesh scale="${scale_ratio} ${scale_ratio} ${scale_ratio}"
-                    filename="file://$(find robot_description)/urdf/meshes/leftwheel.STL" />
-            </geometry>
-        </collision>
+        <!-- <collision>
+            <origin xyz="0 0.03 0" rpy="1.5708 0 0" />
+            <geometry>
+                <cylinder radius="0.082" length="0.06"/>
+            </geometry>
+        </collision> -->
         <xacro:inertial_box mass="1.0582" x="-2.4286E-17" y="-0.033904" z="4.1633E-17">
             <origin xyz="-2.4286E-17 -0.033904 4.1633E-17" rpy="0 0 0" />
@@ -96,8 +105,8 @@
     <!-- Left Wheel Joint -->
     <joint name="leftwheel_joint" type="continuous">
-        <origin xyz="-0.12418 -0.185 -0.063" rpy="0 0 -3.1416" />
+        <origin xyz="-0.12418 -0.185 -0.063" rpy="-${M_PI/2} 0 0" />
         <parent link="base_link" />
         <child link="leftwheel_link" />
-        <axis xyz="0 1 0" />
+        <axis xyz="0 0 1" />
     </joint>
     <!-- Caster Wheel -->
@@ -105,18 +114,20 @@
         <visual>
             <origin xyz="0 0 0" rpy="0 0 0" />
-            <geometry>
-                <mesh scale="${scale_ratio} ${scale_ratio} ${scale_ratio}"
-                    filename="file://$(find robot_description)/urdf/meshes/casterwheel.STL" />
+            <!-- <geometry>
+                <mesh scale="${scale_ratio} ${scale_ratio} ${scale_ratio}"
+                    filename="${path_meshes}/casterwheel.stl" />
+            </geometry> -->
+            <geometry>
+                <cylinder radius="0.04" length="0.02"/>
             </geometry>
             <material name="blue">
             </material>
         </visual>
-        <collision>
-            <origin xyz="0 0 0" rpy="0 0 0" />
-            <geometry>
-                <mesh scale="${scale_ratio} ${scale_ratio} ${scale_ratio}"
-                    filename="file://$(find robot_description)/urdf/meshes/casterwheel.STL" />
-            </geometry>
-        </collision>
+        <!-- <collision>
+            <origin xyz="0 0 0" rpy="1.5708 0 0" />
+            <geometry>
+                <cylinder radius="0.04" length="0.02"/>
+            </geometry>
+        </collision> -->
         <xacro:inertial_box mass="0.10255" x="-0.0032546" y="0.0053327" z="0.013127">
             <origin xyz="-0.0032546 0.0053327 0.013127" rpy="0 0 0" />
@@ -125,5 +136,5 @@
     <!-- Caster Wheel Joint -->
     <joint name="casterwheel_joint" type="fixed">
-        <origin xyz="0.25029 -0.01098 -0.1075" rpy="0 0 0" />
+        <origin xyz="0.25029 -0.01098 -0.1375" rpy="0 0 0" />
         <parent link="base_link" />
         <child link="casterwheel_link" />
@@ -131,16 +142,10 @@
     </joint>
     <!-- Lidar -->
-    <link name="lidar_link">
-        <inertial>
-            <origin xyz="0.00050486 -3.7855E-05 -0.025753" rpy="0 0 0" />
-            <mass value="0.2064" />
-            <inertia ixx="0.00011156" ixy="-1.2701E-07" ixz="-1.6019E-06" iyy="0.00010988"
-                iyz="1.201E-07" izz="0.0001391" />
-        </inertial>
-        <visual>
-            <origin xyz="0 0 0" rpy="0 0 0" />
-            <geometry>
-                <mesh scale="${scale_ratio} ${scale_ratio} ${scale_ratio}"
-                    filename="file://$(find robot_description)/urdf/meshes/lidar.STL" />
+    <!-- <link name="lidar_link">
+        <visual>
+            <origin xyz="0 0 0" rpy="0 0 0" />
+            <geometry>
+                <mesh scale="${scale_ratio} ${scale_ratio} ${scale_ratio}"
+                    filename="${path_meshes}/lidar.STL" />
             </geometry>
             <material name="gray">
@@ -151,5 +156,5 @@
             <geometry>
                 <mesh scale="${scale_ratio} ${scale_ratio} ${scale_ratio}"
-                    filename="file://$(find robot_description)/urdf/meshes/lidar.STL" />
+                    filename="${path_meshes}/lidar.STL" />
             </geometry>
         </collision>
@@ -157,25 +162,19 @@
             <origin xyz="0.00050486 -3.7855E-05 -0.025753" rpy="0 0 0" />
         </xacro:inertial_box>
-    </link>
+    </link> -->
     <!-- Lidar Joint -->
-    <joint name="lidar_joint" type="fixed">
+    <!-- <joint name="lidar_joint" type="fixed">
         <origin xyz="0.00082049 0.00875 0.12332" rpy="0 0 0" />
         <parent link="base_link" />
         <child link="lidar_link" />
         <axis xyz="0 0 1" />
-    </joint>
+    </joint> -->
     <!-- IMU -->
-    <link name="imu_link">
-        <inertial>
-            <origin xyz="-0.015015 -0.00012812 0.00021369" rpy="0 0 0" />
-            <mass value="0.05157" />
-            <inertia ixx="1.5728E-05" ixy="-1.2026E-09" ixz="1.5815E-09" iyy="8.9379E-06"
-                iyz="-2.1887E-10" izz="1.4344E-05" />
-        </inertial>
-        <visual>
-            <origin xyz="0 0 0" rpy="0 0 0" />
-            <geometry>
-                <mesh scale="${scale_ratio} ${scale_ratio} ${scale_ratio}"
-                    filename="file://$(find robot_description)/urdf/meshes/imu.STL" />
+    <!-- <link name="imu_link">
+        <visual>
+            <origin xyz="0 0 0" rpy="0 0 0" />
+            <geometry>
+                <mesh scale="${scale_ratio} ${scale_ratio} ${scale_ratio}"
+                    filename="${path_meshes}/imu.STL" />
             </geometry>
             <material name="black">
@@ -186,5 +185,5 @@
             <geometry>
                 <mesh scale="${scale_ratio} ${scale_ratio} ${scale_ratio}"
-                    filename="file://$(find robot_description)/urdf/meshes/imu.STL" />
+                    filename="${path_meshes}/imu.STL" />
             </geometry>
         </collision>
@@ -192,25 +191,19 @@
             <origin xyz="-0.015015 -0.00012812 0.00021369" rpy="0 0 0" />
         </xacro:inertial_box>
-    </link>
+    </link> -->
     <!-- IMU Joint -->
-    <joint name="imu_joint" type="fixed">
+    <!-- <joint name="imu_joint" type="fixed">
         <origin xyz="0.05082 -0.0047896 0.053918" rpy="0 0 0" />
         <parent link="base_link" />
         <child link="imu_link" />
         <axis xyz="0 0 0" />
-    </joint>
+    </joint> -->
     <!-- Camera -->
-    <link name="camerad435i_link">
-        <inertial>
-            <origin xyz="0.0094812 3.7095E-05 -7.9734E-05" rpy="0 0 0" />
-            <mass value="0.032264" />
-            <inertia ixx="2.2098E-05" ixy="-1.4651E-10" ixz="2.902E-10" iyy="1.9467E-06"
-                iyz="8.3417E-11" izz="2.1858E-05" />
-        </inertial>
-        <visual>
-            <origin xyz="0 0 0" rpy="0 0 0" />
-            <geometry>
-                <mesh scale="${scale_ratio} ${scale_ratio} ${scale_ratio}"
-                    filename="file://$(find robot_description)/urdf/meshes/camerad435i.STL" />
+    <!-- <link name="camerad435i_link">
+        <visual>
+            <origin xyz="0 0 0" rpy="0 0 0" />
+            <geometry>
+                <mesh scale="${scale_ratio} ${scale_ratio} ${scale_ratio}"
+                    filename="${path_meshes}/camerad435i.STL" />
             </geometry>
             <material name="white">
@@ -221,5 +214,5 @@
             <geometry>
                 <mesh scale="${scale_ratio} ${scale_ratio} ${scale_ratio}"
-                    filename="file://$(find robot_description)/urdf/meshes/camerad435i.STL" />
+                    filename="${path_meshes}/camerad435i.STL" />
             </geometry>
         </collision>
@@ -227,25 +220,19 @@
             <origin xyz="0.0094812 3.7095E-05 -7.9734E-05" rpy="0 0 0" />
         </xacro:inertial_box>
-    </link>
+    </link> -->
     <!-- Camera Joint -->
-    <joint name="camerad435i_joint" type="fixed">
+    <!-- <joint name="camerad435i_joint" type="fixed">
         <origin xyz="-0.20718 -0.08268 0.17016" rpy="0 0 0" />
         <parent link="base_link" />
         <child link="camerad435i_link" />
         <axis xyz="0 0 0" />
-    </joint>
+    </joint> -->
     <!-- Camera -->
-    <link name="camerat265_link">
-        <inertial>
-            <origin xyz="0.0061266 3.8568E-05 -1.9004E-05" rpy="0 0 0" />
-            <mass value="0.030988" />
-            <inertia ixx="3.0221E-05" ixy="-1.6541E-10" ixz="4.8935E-11" iyy="1.9363E-06"
-                iyz="9.2265E-11" izz="2.9002E-05" />
-        </inertial>
-        <visual>
-            <origin xyz="0 0 0" rpy="0 0 0" />
-            <geometry>
-                <mesh scale="${scale_ratio} ${scale_ratio} ${scale_ratio}"
-                    filename="file://$(find robot_description)/urdf/meshes/camerat265.STL" />
+    <!-- <link name="camerat265_link">
+        <visual>
+            <origin xyz="0 0 0" rpy="0 0 0" />
+            <geometry>
+                <mesh scale="${scale_ratio} ${scale_ratio} ${scale_ratio}"
+                    filename="${path_meshes}/camerat265.STL" />
             </geometry>
             <material name="white">
@@ -256,5 +243,5 @@
             <geometry>
                 <mesh scale="${scale_ratio} ${scale_ratio} ${scale_ratio}"
-                    filename="file://$(find robot_description)/urdf/meshes/camerat265.STL" />
+                    filename="${path_meshes}/camerat265.STL" />
             </geometry>
         </collision>
@@ -262,11 +249,11 @@
             <origin xyz="0.0061266 3.8568E-05 -1.9004E-05" rpy="0 0 0" />
         </xacro:inertial_box>
-    </link>
+    </link> -->
     <!-- Camera Joint -->
-    <joint name="camerat265_joint" type="fixed">
+    <!-- <joint name="camerat265_joint" type="fixed">
         <origin xyz="-0.20118 0.080908 0.16952" rpy="0 0 0" />
         <parent link="base_link" />
         <child link="camerat265_link" />
         <axis xyz="0 0 0" />
-    </joint>
+    </joint> -->
 </robot>
